Commit message: modify inertial

File: src/snake_robot1/urdf/base_rail1.xacro (robot description, xacro)
@@ -2,4 +2,12 @@
 <robot xmlns:xacro="http://www.ros.org/wiki/xacro" name="base_rail1">
     <xacro:macro name="base1" params="parent *origin name:=base base_joint_type:=prismatic">
+        <xacro:macro name="rail1_default_inertial">
+            <inertial>
+                    <mass value="0.024744" />
+                    <inertia ixx="0.000017" ixy="0.0" ixz="0.0"
+                            iyy="0.000016" iyz="0.0"
+                            izz="0.000028" />
+            </inertial>
+        </xacro:macro>
         <link
             name="${name}_link">
@@ -48,18 +56,5 @@
         <link
         name="${name}_link1">
-        <inertial>
-        <origin
-            xyz="7.2882E-09 3.4329E-09 0.010539"
-            rpy="0 0 0" />
-        <mass
-            value="0.024744" />
-        <inertia
-            ixx="1.4926E-05"
-            ixy="-1.6133E-09"
-            ixz="2.3902E-13"
-            iyy="1.4062E-05"
-            iyz="-9.0592E-13"
-            izz="2.7906E-05" />
-        </inertial>
+        <xacro:rail1_default_inertial/>
         <visual>
         <origin
@@ -104,18 +99,5 @@
     <link
         name="${name}_link2">
-        <inertial>
-        <origin
-            xyz="-3.433E-09 7.2882E-09 0.010539"
-            rpy="0 0 0" />
-        <mass
-            value="0.024744" />
-        <inertia
-            ixx="1.4062E-05"
-            ixy="1.6133E-09"
-            ixz="9.0592E-13"
-            iyy="1.4926E-05"
-            iyz="2.3902E-13"
-            izz="2.7906E-05" />
-        </inertial>
+        <xacro:rail1_default_inertial/>
         <visual>
         <origin
@@ -162,18 +144,5 @@
     <link
         name="${name}_link3">
-        <inertial>
-        <origin
-            xyz="7.2882E-09 3.4329E-09 0.010539"
-            rpy="0 0 0" />
-        <mass
-            value="0.024744" />
-        <inertia
-            ixx="1.4926E-05"
-            ixy="-1.6133E-09"
-            ixz="2.3902E-13"
-            iyy="1.4062E-05"
-            iyz="-9.0592E-13"
-            izz="2.7906E-05" />
-        </inertial>
+        <xacro:rail1_default_inertial/>
         <visual>
         <origin
@@ -220,18 +189,5 @@
     <link
         name="${name}_link4">
-        <inertial>
-        <origin
-            xyz="-3.433E-09 7.2882E-09 0.010539"
-            rpy="0 0 0" />
-        <mass
-            value="0.024744" />
-        <inertia
-            ixx="1.4062E-05"
-            ixy="1.6133E-09"
-            ixz="9.0592E-13"
-            iyy="1.4926E-05"
-            iyz="2.3902E-13"
-            izz="2.7906E-05" />
-        </inertial>
+        <xacro:rail1_default_inertial/>
         <visual>
         <origin
@@ -278,18 +234,5 @@
     <link
         name="${name}_link5">
-        <inertial>
-        <origin
-            xyz="7.2882E-09 3.4329E-09 0.010539"
-            rpy="0 0 0" />
-        <mass
-            value="0.024744" />
-        <inertia
-            ixx="1.4926E-05"
-            ixy="-1.6133E-09"
-            ixz="2.3902E-13"
-            iyy="1.4062E-05"
-            iyz="-9.0592E-13"
-            izz="2.7906E-05" />
-        </inertial>
+        <xacro:rail1_default_inertial/>
         <visual>
         <origin

File: src/snake_robot2/urdf/base_rail2.xacro (robot description, xacro)
@@ -2,4 +2,12 @@
 <robot xmlns:xacro="http://www.ros.org/wiki/xacro" name="base_rail2">
   <xacro:macro name="base2" params="parent *origin name:=base base_joint_type:=prismatic">
+    <xacro:macro name="rail2_default_inertial">
+        <inertial>
+                <mass value="0.018285" />
+                <inertia ixx="0.000008" ixy="0.0" ixz="0.0"
+                      iyy="0.000007" iyz="0.0"
+                      izz="0.000010" />
+        </inertial>
+    </xacro:macro>
     <link
       name="${name}_link">
@@ -48,18 +56,5 @@
     <link
       name="${name}_link1">
-      <inertial>
-        <origin
-          xyz="5.5313E-09 3.6738E-09 0.010533"
-          rpy="0 0 0" />
-        <mass
-          value="0.018285" />
-        <inertia
-          ixx="5.7939E-06"
-          ixy="-9.0258E-10"
-          ixz="-4.854E-14"
-          iyy="5.3329E-06"
-          iyz="-9.0945E-13"
-          izz="1.0221E-05" />
-      </inertial>
+      <xacro:rail2_default_inertial/>
       <visual>
         <origin
@@ -104,18 +99,5 @@
     <link
       name="${name}_link2">
-      <inertial>
-        <origin
-          xyz="-3.6738E-09 5.5318E-09 0.010533"
-          rpy="0 0 0" />
-        <mass
-          value="0.018285" />
-        <inertia
-          ixx="5.3329E-06"
-          ixy="9.0258E-10"
-          ixz="9.0945E-13"
-          iyy="5.7939E-06"
-          iyz="-4.854E-14"
-          izz="1.0221E-05" />
-      </inertial>
+      <xacro:rail2_default_inertial/>
       <visual>
         <origin
@@ -162,18 +144,5 @@
     <link
       name="${name}_link3">
-      <inertial>
-        <origin
-          xyz="5.5313E-09 3.6738E-09 0.010533"
-          rpy="0 0 0" />
-        <mass
-          value="0.018285" />
-        <inertia
-          ixx="5.7939E-06"
-          ixy="-9.0258E-10"
-          ixz="-4.854E-14"
-          iyy="5.3329E-06"
-          iyz="-9.0945E-13"
-          izz="1.0221E-05" />
-      </inertial>
+      <xacro:rail2_default_inertial/>
       <visual>
         <origin
@@ -220,18 +189,5 @@
     <link
       name="${name}_link4">
-      <inertial>
-        <origin
-          xyz="-3.6738E-09 5.5318E-09 0.010533"
-          rpy="0 0 0" />
-        <mass
-          value="0.018285" />
-        <inertia
-          ixx="5.3329E-06"
-          ixy="9.0258E-10"
-          ixz="9.0945E-13"
-          iyy="5.7939E-06"
-          iyz="-4.854E-14"
-          izz="1.0221E-05" />
-      </inertial>
+      <xacro:rail2_default_inertial/>
       <visual>
         <origin
@@ -278,18 +234,5 @@
     <link
       name="${name}_link5">
-      <inertial>
-        <origin
-          xyz="5.5313E-09 3.6738E-09 0.010533"
-          rpy="0 0 0" />
-        <mass
-          value="0.018285" />
-        <inertia
-          ixx="5.7939E-06"
-          ixy="-9.0258E-10"
-          ixz="-4.854E-14"
-          iyy="5.3329E-06"
-          iyz="-9.0945E-13"
-          izz="1.0221E-05" />
-      </inertial>
+      <xacro:rail2_default_inertial/>
       <visual>
         <origin
